File: BABY_Kicad/BABY_Kicad.kicad_pcb (KiCad board)
At the start: 2 copper layers, 139 x 128.5 mm, 113 parts, among them J1 Reset, J10 Con4_Top, J11 Con2_Bottom, J12 Con3_Bottom, J13 Con4_Bottom, J2 Clock_in, J3 Gate_Out, J4 CV, J6 Con1_Top, J7 Con1_Bottom, J8 Con2_Top, J9 Con3_Top, Q1 2N3904, Q2 2N3904, Q3 2N3904, Q4 2N3904, Q5 2N3904, Q6 BC548, SW1 Gate1, SW2 Gate2, SW3 Gate3, SW4 Gate4, SW5 Gate5, SW6 SW_DPDT_x2, SW7 SW_DPDT_x2, U1 4017, U2 TL074

Commit message: finished pcb
Parts:
- removed R28, R29, R30, R31, R32: 1k, 2_BenjiaoFootprints:Resistor_L6.3mm_D2.5mm_P7.62mm_Horizontal
- C1, C3, J5, RV1, RV7, RV8: moved to B.Cu
- Q1, Q2, Q3, Q4, Q5, Q6: footprint Package_TO_SOT_THT:TO-92_Inline -> Package_TO_SOT_THT:TO-92_Wide
- moved RV7 153.1 mm to (125.1, 51.3)
- moved RV8 152.0 mm to (125.2, 56.7)
- moved RV1 151.3 mm to (125.2, 45.5)
- moved J5 133.8 mm to (130.2, 106.0), turned to 180 degrees
- moved C1 132.2 mm to (143.6, 103.7), turned to 180 degrees
- moved R14 129.4 mm to (129.0, 68.1), turned to 180 degrees
- moved C3 128.0 mm to (148.6, 108.0), turned to 180 degrees
- moved R4 115.1 mm to (121.5, 61.7)
- moved R33 110.2 mm to (132.0, 55.9), turned to 0 degrees
- moved R3 108.5 mm to (129.0, 65.0), turned to 180 degrees
- moved R18 105.7 mm to (146.4, 72.5), turned to -90 degrees
- moved D18 105.6 mm to (132.2, 113.0), turned to 180 degrees
- moved R38 103.7 mm to (129.1, 74.0), turned to 180 degrees
- moved D7 103.5 mm to (123.8, 83.2), turned to -90 degrees
- moved D19 103.2 mm to (135.9, 113.0)
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- renumbered REF** to REF1, REF** to REF10, REF** to REF11, REF** to REF12, REF** to REF13, REF** to REF14, REF** to REF15, REF** to REF16, REF** to REF17, REF** to REF2, REF** to REF3, REF** to REF4, REF** to REF5, REF** to REF6, REF** to REF7, REF** to REF8, REF** to REF9
Connections:
- C2 pad 1: Net-(C2-Pad1) -> 22_B
- D1 pad 1: Net-(D1-K) -> 16_T
- D1 pad 2: 12V -> 12V_T
- D10 pad 2: Net-(D10-A) -> 3_B
- D11 pad 2: Net-(D11-A) -> 4_B
- D12 pad 2: Net-(D12-A) -> 5_B
- D13 pad 2: Net-(D13-A) -> 6_B
- D14 pad 2: Net-(D14-A) -> 7_B
- D15 pad 2: Net-(D15-A) -> 8_B
- D16 pad 2: Net-(D16-A) -> 9_B
- D17 pad 2: Net-(D17-A) -> 10_B
- D2 pad 1: Net-(D2-K) -> 17_T
- D2 pad 2: 12V -> 12V_T
- D21 pad 2: Net-(D21-A) -> 15_B
- D3 pad 1: Net-(D3-K) -> 18_T
- D3 pad 2: 12V -> 12V_T
- D4 pad 1: Net-(D4-K) -> 19_T
- D4 pad 2: 12V -> 12V_T
- D5 pad 1: Net-(D5-K) -> 20_T
- D5 pad 2: 12V -> 12V_T
- D7 pad 2: Net-(D7-A) -> 24_B
- D8 pad 2: Net-(D8-A) -> 1_B
- D9 pad 2: Net-(D9-A) -> 2_B
- J1 pad S: GND -> GND_T
- J1 pad T: Net-(C2-Pad1) -> 22_T
- J10 pad 1: unconnected-(J10-Pin_1-Pad1) -> 20_T
- J10 pad 10: unconnected-(J10-Pin_10-Pad10) -> GND_T
- J10 pad 11: unconnected-(J10-Pin_11-Pad11) -> GND_T
- J10 pad 12: unconnected-(J10-Pin_12-Pad12) -> GND_T
- J10 pad 13: unconnected-(J10-Pin_13-Pad13) -> GND_T
- J10 pad 14: unconnected-(J10-Pin_14-Pad14) -> GND_T
- J10 pad 2: unconnected-(J10-Pin_2-Pad2) -> 19_T
- J10 pad 3: unconnected-(J10-Pin_3-Pad3) -> 18_T
- J10 pad 4: unconnected-(J10-Pin_4-Pad4) -> 17_T
- J10 pad 5: unconnected-(J10-Pin_5-Pad5) -> 16_T
- J10 pad 6: unconnected-(J10-Pin_6-Pad6) -> 21_T
- J10 pad 7: unconnected-(J10-Pin_7-Pad7) -> GND_T
- J10 pad 8: unconnected-(J10-Pin_8-Pad8) -> GND_T
- J10 pad 9: unconnected-(J10-Pin_9-Pad9) -> GND_T
- J11 pad 1: unconnected-(J11-Pin_1-Pad1) -> 12_B
- J11 pad 10: unconnected-(J11-Pin_10-Pad10) -> 28_B
- J11 pad 2: unconnected-(J11-Pin_2-Pad2) -> 13_B
- J11 pad 3: unconnected-(J11-Pin_3-Pad3) -> 14_B
- J11 pad 4: unconnected-(J11-Pin_4-Pad4) -> 11_B
- J11 pad 5: unconnected-(J11-Pin_5-Pad5) -> 15_B
- J11 pad 6: unconnected-(J11-Pin_6-Pad6) -> 22_B
- J11 pad 7: unconnected-(J11-Pin_7-Pad7) -> 26_B
- J11 pad 8: unconnected-(J11-Pin_8-Pad8) -> 25_B
- J11 pad 9: unconnected-(J11-Pin_9-Pad9) -> 27_B
- J12 pad 1: unconnected-(J12-Pin_1-Pad1) -> 23_B
- J12 pad 10: unconnected-(J12-Pin_10-Pad10) -> 29_B
- J12 pad 2: unconnected-(J12-Pin_2-Pad2) -> 24_B
- J12 pad 3: unconnected-(J12-Pin_3-Pad3) -> 12V
- J12 pad 4: unconnected-(J12-Pin_4-Pad4) -> 35_B
- J12 pad 5: unconnected-(J12-Pin_5-Pad5) -> 30_B
- J12 pad 6: unconnected-(J12-Pin_6-Pad6) -> 31_B
- J12 pad 7: unconnected-(J12-Pin_7-Pad7) -> 32_B
- J12 pad 8: unconnected-(J12-Pin_8-Pad8) -> 33_B
- J12 pad 9: unconnected-(J12-Pin_9-Pad9) -> 34_B
- J13 pad 1: unconnected-(J13-Pin_1-Pad1) -> 20_B
- J13 pad 10: unconnected-(J13-Pin_10-Pad10) -> GND
- J13 pad 11: unconnected-(J13-Pin_11-Pad11) -> GND
- J13 pad 12: unconnected-(J13-Pin_12-Pad12) -> GND
- J13 pad 13: unconnected-(J13-Pin_13-Pad13) -> GND
- J13 pad 14: unconnected-(J13-Pin_14-Pad14) -> GND
- J13 pad 2: unconnected-(J13-Pin_2-Pad2) -> 19_B
- J13 pad 3: unconnected-(J13-Pin_3-Pad3) -> 18_B
- J13 pad 4: unconnected-(J13-Pin_4-Pad4) -> 17_B
- J13 pad 5: unconnected-(J13-Pin_5-Pad5) -> 16_B
- J13 pad 6: unconnected-(J13-Pin_6-Pad6) -> 21_B
- J13 pad 7: unconnected-(J13-Pin_7-Pad7) -> GND
- J13 pad 8: unconnected-(J13-Pin_8-Pad8) -> GND
- J13 pad 9: unconnected-(J13-Pin_9-Pad9) -> GND
- J2 pad S: GND -> GND_T
- J2 pad T: Net-(D21-A) -> 15_T
- J3 pad S: GND -> GND_T
- J3 pad T: Net-(J3-PadT) -> 21_T
- J4 pad S: GND -> GND_T
- J4 pad T: Net-(J4-PadT) -> 23_T
- J6 pad 1: unconnected-(J6-Pin_1-Pad1) -> 10_T
- J6 pad 10: unconnected-(J6-Pin_10-Pad10) -> 1_T
- J6 pad 2: unconnected-(J6-Pin_2-Pad2) -> 9_T
- J6 pad 3: unconnected-(J6-Pin_3-Pad3) -> 8_T
- J6 pad 4: unconnected-(J6-Pin_4-Pad4) -> 7_T
- J6 pad 5: unconnected-(J6-Pin_5-Pad5) -> 6_T
- J6 pad 6: unconnected-(J6-Pin_6-Pad6) -> 5_T
- J6 pad 7: unconnected-(J6-Pin_7-Pad7) -> 4_T
- J6 pad 8: unconnected-(J6-Pin_8-Pad8) -> 3_T
- J6 pad 9: unconnected-(J6-Pin_9-Pad9) -> 2_T
- J7 pad 1: unconnected-(J7-Pin_1-Pad1) -> 10_B
- J7 pad 10: unconnected-(J7-Pin_10-Pad10) -> 1_B
- J7 pad 2: unconnected-(J7-Pin_2-Pad2) -> 9_B
- J7 pad 3: unconnected-(J7-Pin_3-Pad3) -> 8_B
- J7 pad 4: unconnected-(J7-Pin_4-Pad4) -> 7_B
- J7 pad 5: unconnected-(J7-Pin_5-Pad5) -> 6_B
- J7 pad 6: unconnected-(J7-Pin_6-Pad6) -> 5_B
- J7 pad 7: unconnected-(J7-Pin_7-Pad7) -> 4_B
- J7 pad 8: unconnected-(J7-Pin_8-Pad8) -> 3_B
- J7 pad 9: unconnected-(J7-Pin_9-Pad9) -> 2_B
- J8 pad 1: unconnected-(J8-Pin_1-Pad1) -> 12_T
- J8 pad 10: unconnected-(J8-Pin_10-Pad10) -> 28_T
- J8 pad 2: unconnected-(J8-Pin_2-Pad2) -> 13_T
- J8 pad 3: unconnected-(J8-Pin_3-Pad3) -> 14_T
- J8 pad 4: unconnected-(J8-Pin_4-Pad4) -> 11_T
- J8 pad 5: unconnected-(J8-Pin_5-Pad5) -> 15_T
- J8 pad 6: unconnected-(J8-Pin_6-Pad6) -> 22_T
- J8 pad 7: unconnected-(J8-Pin_7-Pad7) -> 26_T
- J8 pad 8: unconnected-(J8-Pin_8-Pad8) -> 25_T
- J8 pad 9: unconnected-(J8-Pin_9-Pad9) -> 27_T
- J9 pad 1: unconnected-(J9-Pin_1-Pad1) -> 23_T
- J9 pad 10: unconnected-(J9-Pin_10-Pad10) -> 29_T
- J9 pad 2: unconnected-(J9-Pin_2-Pad2) -> 24_T
- J9 pad 3: unconnected-(J9-Pin_3-Pad3) -> 12V_T
- J9 pad 4: unconnected-(J9-Pin_4-Pad4) -> 35_T
- J9 pad 5: unconnected-(J9-Pin_5-Pad5) -> 25_T
- J9 pad 6: unconnected-(J9-Pin_6-Pad6) -> 26_T
- J9 pad 7: unconnected-(J9-Pin_7-Pad7) -> 27_T
- J9 pad 8: unconnected-(J9-Pin_8-Pad8) -> 28_T
- J9 pad 9: unconnected-(J9-Pin_9-Pad9) -> 29_T
- R11 pad 2: Net-(D4-K) -> 19_B
- R12 pad 2: Net-(D5-K) -> 20_B
- R23 pad 1: Net-(SW1-A) -> 25_B
- R24 pad 1: Net-(SW2-A) -> 26_B
- R25 pad 1: Net-(SW3-A) -> 27_B
- R26 pad 1: Net-(SW4-A) -> 28_B
- R27 pad 1: Net-(SW5-A) -> 29_B
- R3 pad 2: Net-(SW7A-A) -> 12_B
- R33 pad 2: Net-(SW7A-B) -> 11_B
- R38 pad 2: Net-(J4-PadT) -> 23_B
- R4 pad 1: Net-(SW7B-A) -> 13_B
- R5 pad 2: Net-(SW7B-C) -> 14_B
- R6 pad 2: Net-(D1-K) -> 16_B
- R7 pad 1: Net-(J3-PadT) -> 21_B
- R8 pad 2: Net-(D2-K) -> 17_B
- R9 pad 2: Net-(D3-K) -> 18_B
- RV1 pad 1: Net-(R3-Pad1) -> GND
- RV1 pad 3: GND -> Net-(R3-Pad1)
- RV2 pad 1: GND -> GND_T
- RV2 pad 2: Net-(D13-A) -> 6_T
- RV2 pad 3: Net-(SW1-A) -> 25_T
- RV3 pad 1: GND -> GND_T
- RV3 pad 2: Net-(D14-A) -> 7_T
- RV3 pad 3: Net-(SW2-A) -> 26_T
- RV4 pad 1: GND -> GND_T
- RV4 pad 2: Net-(D15-A) -> 8_T
- RV4 pad 3: Net-(SW3-A) -> 27_T
- RV5 pad 1: GND -> GND_T
- RV5 pad 2: Net-(D16-A) -> 9_T
- RV5 pad 3: Net-(SW4-A) -> 28_T
- RV6 pad 1: GND -> GND_T
- RV6 pad 2: Net-(D17-A) -> 10_T
- RV6 pad 3: Net-(SW5-A) -> 29_T
- SW1 pad 1: Net-(SW1-A) -> 25_T
- SW1 pad 2: Net-(D8-A) -> 1_T
- SW2 pad 1: Net-(SW2-A) -> 26_T
- SW2 pad 2: Net-(D9-A) -> 2_T
- SW3 pad 1: Net-(SW3-A) -> 27_T
- SW3 pad 2: Net-(D10-A) -> 3_T
- SW4 pad 1: Net-(SW4-A) -> 28_T
- SW4 pad 2: Net-(D11-A) -> 4_T
- SW5 pad 1: Net-(SW5-A) -> 29_T
- SW5 pad 2: Net-(D12-A) -> 5_T
- SW6 pad 1: Net-(SW4-A) -> 28_T
- SW6 pad 2: Net-(D7-A) -> 24_T
- SW6 pad 4: Net-(SW5-A) -> 29_T
- SW6 pad 6: Net-(SW6B-C) -> 35_T
- SW7 pad 1: Net-(SW7A-A) -> 12_T
- SW7 pad 2: Net-(SW7A-B) -> 11_T
- SW7 pad 4: Net-(SW7B-A) -> 13_T
- SW7 pad 6: Net-(SW7B-C) -> 14_T
- U1 pad 1: Net-(SW6B-C) -> 35_B
- U1 pad 10: Net-(SW5-A) -> 34_B
- U1 pad 2: Net-(SW2-A) -> 31_B
- U1 pad 3: Net-(SW1-A) -> 30_B
- U1 pad 4: Net-(SW3-A) -> 32_B
- U1 pad 7: Net-(SW4-A) -> 33_B
- U2 pad 12: Net-(SW7A-B) -> 11_B
Routing:
- net GND: track 0.00 -> 267.5 mm, vias 0 -> 1
- net GND_T: track 0.00 -> 192.0 mm
- net 10_T: track 0.00 -> 124.4 mm, vias 0 -> 1
- net 12V_T: track 0.00 -> 114.9 mm
- net 12V: track 0.00 -> 102.2 mm
- net 5_T: track 0.00 -> 97.8 mm
- net 25_T: track 0.00 -> 97.6 mm, vias 0 -> 1
- net 29_T: track 0.00 -> 96.4 mm, vias 0 -> 1
- net 9_T: track 0.00 -> 92.1 mm
- net 16_T: track 0.00 -> 89.4 mm
- net -12V: track 0.00 -> 76.1 mm
- net Net-(D20-K): track 0.00 -> 72.1 mm, vias 0 -> 1
- net 17_T: track 0.00 -> 69.2 mm, vias 0 -> 1
- net 4_T: track 0.00 -> 66.8 mm
- net 35_B: track 0.00 -> 66.5 mm, vias 0 -> 1
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
Commit message: first testrun
Parts:
- added R99: 0, Resistor_SMD:R_0201_0603Metric, B.Cu at (21.1, 28.6)
- added Ref**: Val**, 3_Graphics:logo_v1, F.Cu at (43.2, 149.6)
Routing:
- net Net-(R99-Pad1): vias 0 -> 1
- added copper zone on B.Cu, net Net-(R99-Pad1)
- added copper zone on F.Cu, net Net-(R99-Pad1)
Other:
- board text added: "1v"
- board text added: "2v"
- board text added: "5v"
- board text added: "JLCJLCJLCJLC"
- board text added: "Oh Baby 1.0 Control March 23"
- board text added: "Oh Baby 1.0 Main March 23"
- board text added: "OhBaby 1.0 March 23 Panel"
- board text added: "Top Side, Bottom"
- board text added: "Top orientation, bottom end here"

Commit message: Fixes
Parts:
- moved D1 2.53 mm to (102.7, 61.6), turned to 0 degrees
Connections:
- SW6 pad 1: 28_T -> 29_T
- SW6 pad 2: 24_T -> Net-(SW6A-B)
- SW6 pad 3: Net-(SW6A-C) -> 35_T
- SW6 pad 4: 29_T -> 28_T
- SW6 pad 5: Net-(SW6A-C) -> 24_T
- SW6 pad 6: 35_T -> Net-(SW6A-B)
- SW7 pad 1: 12_T -> 13_T
- SW7 pad 2: 11_T -> Net-(SW7A-B)
- SW7 pad 3: Net-(SW7A-C) -> 14_T
- SW7 pad 4: 13_T -> 12_T
- SW7 pad 5: Net-(SW7A-C) -> 11_T
- SW7 pad 6: 14_T -> Net-(SW7A-B)
Routing:
- net 11_T: track 10.0 -> 32.3 mm
- net 28_T: track 59.8 -> 70.3 mm
- net Net-(SW7A-C): track 8.76 -> 0.00 mm
- net 35_T: track 50.0 -> 58.5 mm, vias 0 -> 1
- net Net-(SW6A-C): track 8.35 -> 0.00 mm
- net Net-(SW6A-B): track 0.00 -> 6.79 mm
- net Net-(SW7A-B): track 0.00 -> 6.79 mm
- net 16_T: track 89.4 -> 95.3 mm
- net 12_T: track 8.75 -> 4.27 mm
- net 24_T: track 47.1 -> 43.0 mm
- net 29_T: track 96.4 -> 92.5 mm
- net 26_T: track 65.4 -> 67.0 mm
- net GND_T: track 192.0 -> 193.4 mm
- net 12V_T: track 114.9 -> 113.8 mm
- net 13_T: track 4.43 -> 5.21 mm
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Other:
- board text added: "New: SW6/7 type 1 ON-ON-ON"
- board text added: "Oh Baby 1.1 Control Works with 1.0 Main"
- board text added: "OhBaby 1.1 March 23 Panel Fixed Switch Hole Size"
- board text removed: "Oh Baby 1.0 Control March 23"
- board text removed: "OhBaby 1.0 March 23 Panel"
