File: BABY_Kicad/BABY_Kicad.kicad_sch (KiCad schematic)
At the start: 83 parts, among them J1 Reset, J2 Clock_in, J3 Gate_Out, J4 CV, Q1 2N3904, Q2 2N3904, Q3 2N3904, Q4 2N3904, Q5 2N3904, Q6 BC548, SW1 Gate1, SW2 Gate2, SW3 Gate3, SW4 Gate4, SW5 Gate5, SW6 SW_DPDT_x2, SW7 SW_DPDT_x2, U1 4017, U2 TL074

Commit message: started pcb
Parts:
- removed R28, R29, R30, R31, R32: 1k, 2_BenjiaoFootprints:Resistor_L6.3mm_D2.5mm_P7.62mm_Horizontal, symbol Device:R
- added J10: Con4_Top, Connector_PinHeader_2.54mm:PinHeader_1x14_P2.54mm_Vertical, symbol Connector:Conn_01x14_Pin
- added J11: Con2_Bottom, Connector_PinHeader_2.54mm:PinHeader_1x10_P2.54mm_Vertical, symbol Connector:Conn_01x10_Socket
- added J12: Con3_Bottom, Connector_PinHeader_2.54mm:PinHeader_1x10_P2.54mm_Vertical, symbol Connector:Conn_01x10_Socket
- added J13: Con4_Bottom, Connector_PinHeader_2.54mm:PinHeader_1x14_P2.54mm_Vertical, symbol Connector:Conn_01x14_Socket
- added J6: Con1_Top, Connector_PinHeader_2.54mm:PinHeader_1x10_P2.54mm_Vertical, symbol Connector:Conn_01x10_Pin
- added J7: Con1_Bottom, Connector_PinHeader_2.54mm:PinHeader_1x10_P2.54mm_Vertical, symbol Connector:Conn_01x10_Socket
- added J8: Con2_Top, Connector_PinHeader_2.54mm:PinHeader_1x10_P2.54mm_Vertical, symbol Connector:Conn_01x10_Pin
- added J9: Con3_Top, Connector_PinHeader_2.54mm:PinHeader_1x10_P2.54mm_Vertical, symbol Connector:Conn_01x10_Pin
- added R11, R12, R6, R8, R9: 1k, 2_BenjiaoFootprints:Resistor_L6.3mm_D2.5mm_P7.62mm_Horizontal, symbol Device:R
- SW6, SW7: footprint (none) -> 1_SynthFootprints:DPDT_Tayda
Connections:
- net 12V: now also D1.2 (A), D2.2 (A), D3.2 (A), D4.2 (A), D5.2 (A)
- net at Q5.3 (C): now also R12.1; no longer D5.1 (K)
- net at Q1.3 (C): now also R6.1; no longer D1.1 (K)
- net at Q2.3 (C): now also R8.1; no longer D2.1 (K)
- net at Q4.3 (C): now also R11.1; no longer D4.1 (K)
- net at D3.1 (K): now also R9.2; no longer Q3.3 (C)
- new net: D4.1 (K), R11.2
- new net: D2.1 (K), R8.2
- new net: D5.1 (K), R12.2
- new net: D1.1 (K), R6.2
- new net: Q3.3 (C), R9.1
Other:
- moved on the sheet: D4

Commit message: finished pcb
Parts:
- Q1, Q2, Q3, Q4, Q5, Q6: footprint Package_TO_SOT_THT:TO-92_Inline -> Package_TO_SOT_THT:TO-92_Wide
Connections:
- net 12V: now also J12.3 (Pin_3); no longer D1.2 (A), D2.2 (A), D3.2 (A), D4.2 (A), D5.2 (A)
- net GND: now also J13.10 (Pin_10), J13.11 (Pin_11), J13.12 (Pin_12), J13.13 (Pin_13), J13.14 (Pin_14), J13.7 (Pin_7), J13.8 (Pin_8), J13.9 (Pin_9), RV1.1; no longer J1.S, J2.S, J3.S, J4.S, RV1.3, RV2.1, RV3.1, RV4.1, RV5.1, RV6.1
- net 19_B: now reaches R11.2
- net 19_B: now also J13.2 (Pin_2); no longer D4.1 (K)
- net 29_T: now reaches RV6.3, SW5.1 (A), SW6.4 (A)
- net 29_T: now also J9.10 (Pin_10), J9.9 (Pin_9); no longer R27.1, U1.10 (Q4)
- net 17_B: now reaches R8.2
- net 17_B: now also J13.4 (Pin_4); no longer D2.1 (K)
- net at R3.1: now also RV1.3; no longer RV1.1
- net 26_T: now reaches RV3.3, SW2.1 (A)
- net 26_T: now also J8.7 (Pin_7), J9.6 (Pin_6); no longer R24.1, U1.2 (Q1)
- net 2_B: now reaches D9.2 (A)
- net 2_B: now also J7.9 (Pin_9); no longer SW2.2 (B)
- net 24_B: now reaches D7.2 (A)
- net 24_B: now also J12.2 (Pin_2); no longer SW6.2 (B)
- net 22_B: now reaches C2.1
- net 22_B: now also J11.6 (Pin_6); no longer J1.T
- net 20_B: now reaches R12.2
- net 20_B: now also J13.1 (Pin_1); no longer D5.1 (K)
- net 28_T: now reaches RV5.3, SW4.1 (A), SW6.1 (A)
- net 28_T: now also J8.10 (Pin_10), J9.8 (Pin_8); no longer R26.1, U1.7 (Q3)
- net 4_B: now reaches D11.2 (A)
- net 4_B: now also J7.7 (Pin_7); no longer SW4.2 (B)
- net 11_B: now reaches R33.2, U2.12 (+)
- net 11_B: now also J11.4 (Pin_4); no longer SW7.2 (B)
- net 7_B: now reaches D14.2 (A)
- net 7_B: now also J7.4 (Pin_4); no longer RV3.2
- net 3_B: now reaches D10.2 (A)
- net 3_B: now also J7.8 (Pin_8); no longer SW3.2 (B)
- net 18_B: now reaches J13.3 (Pin_3)
- net 18_B: now also R9.2
- net 16_B: now reaches J13.5 (Pin_5)
- net 16_B: now also R6.2
- net 21_B: now reaches J13.6 (Pin_6)
- net 21_B: now also R7.1
- net 16_T: now reaches D1.1 (K)
- net 16_T: now also J10.5 (Pin_5); no longer R6.2
- net 20_T: now reaches J10.1 (Pin_1)
- net 20_T: now also D5.1 (K)
- net GND_T: now reaches J10.10 (Pin_10)
- net GND_T: now also J1.S, J10.11 (Pin_11), J10.12 (Pin_12), J10.13 (Pin_13), J10.14 (Pin_14), J10.7 (Pin_7), J10.8 (Pin_8), J10.9 (Pin_9), J2.S, J3.S, J4.S, RV2.1, RV3.1, RV4.1, RV5.1, RV6.1
- net 19_T: now reaches J10.2 (Pin_2)
- net 19_T: now also D4.1 (K)
- net 18_T: now reaches J10.3 (Pin_3)
- net 18_T: now also D3.1 (K)
- net 17_T: now reaches J10.4 (Pin_4)
- net 17_T: now also D2.1 (K)
- net 21_T: now reaches J10.6 (Pin_6)
- net 21_T: now also J3.T
- net 23_T: now reaches J9.1 (Pin_1)
- net 23_T: now also J4.T
- net 24_T: now reaches J9.2 (Pin_2)
- net 24_T: now also SW6.2 (B)
- net 12V_T: now reaches J9.3 (Pin_3)
- net 12V_T: now also D1.2 (A), D2.2 (A), D3.2 (A), D4.2 (A), D5.2 (A)
- net 35_T: now reaches J9.4 (Pin_4)
- net 35_T: now also SW6.6 (C)
- net 25_T: now reaches J9.5 (Pin_5)
- net 25_T: now also J8.8 (Pin_8), RV2.3, SW1.1 (A)
- net 27_T: now reaches J9.7 (Pin_7)
- net 27_T: now also J8.9 (Pin_9), RV4.3, SW3.1 (A)
- net 15_B: now reaches D21.2 (A)
- net 15_B: now also J11.5 (Pin_5); no longer J2.T
- net 1_B: now reaches D8.2 (A)
- net 1_B: now also J7.10 (Pin_10); no longer SW1.2 (B)
- net 10_B: now reaches D17.2 (A)
- net 10_B: now also J7.1 (Pin_1); no longer RV6.2
- net 6_B: now reaches D13.2 (A)
- net 6_B: now also J7.5 (Pin_5); no longer RV2.2
- net 5_B: now reaches D12.2 (A)
- net 5_B: now also J7.6 (Pin_6); no longer SW5.2 (B)
- net 8_B: now reaches D15.2 (A)
- net 8_B: now also J7.3 (Pin_3); no longer RV4.2
- net 13_B: now reaches R4.1
- net 13_B: now also J11.2 (Pin_2); no longer SW7.4 (A)
- net 14_B: now reaches R5.2
- net 14_B: now also J11.3 (Pin_3); no longer SW7.6 (C)
- net 9_B: now reaches D16.2 (A)
- net 9_B: now also J7.2 (Pin_2); no longer RV5.2
- net 12_B: now reaches J11.1 (Pin_1)
- net 12_B: now also R3.2
- net 28_B: now reaches J11.10 (Pin_10)
- net 28_B: now also R26.1
- net 26_B: now reaches J11.7 (Pin_7)
- net 26_B: now also R24.1
- net 25_B: now reaches J11.8 (Pin_8)
- net 25_B: now also R23.1
- net 27_B: now reaches J11.9 (Pin_9)
- net 27_B: now also R25.1
- net 12_T: now reaches SW7.1 (A)
- net 12_T: now also J8.1 (Pin_1); no longer R3.2
- net 13_T: now reaches J8.2 (Pin_2)
- net 13_T: now also SW7.4 (A)
- net 14_T: now reaches J8.3 (Pin_3)
- net 14_T: now also SW7.6 (C)
- net 11_T: now reaches J8.4 (Pin_4)
- net 11_T: now also SW7.2 (B)
- net 15_T: now reaches J8.5 (Pin_5)
- net 15_T: now also J2.T
- net 22_T: now reaches J8.6 (Pin_6)
- net 22_T: now also J1.T
- net 10_T: now reaches J6.1 (Pin_1)
- net 10_T: now also RV6.2
- net 1_T: now reaches J6.10 (Pin_10)
- net 1_T: now also SW1.2 (B)
- net 9_T: now reaches J6.2 (Pin_2)
- net 9_T: now also RV5.2
- net 8_T: now reaches J6.3 (Pin_3)
- net 8_T: now also RV4.2
- net 7_T: now reaches J6.4 (Pin_4)
- net 7_T: now also RV3.2
- net 6_T: now reaches J6.5 (Pin_5)
- net 6_T: now also RV2.2
- net 5_T: now reaches J6.6 (Pin_6)
- net 5_T: now also SW5.2 (B)
- net 4_T: now reaches J6.7 (Pin_7)
- net 4_T: now also SW4.2 (B)
- net 3_T: now reaches J6.8 (Pin_8)
- net 3_T: now also SW3.2 (B)
- net 2_T: now reaches J6.9 (Pin_9)
- net 2_T: now also SW2.2 (B)
- net 35_B: now reaches U1.1 (Q5)
- net 35_B: now also J12.4 (Pin_4); no longer SW6.6 (C)
- net 23_B: now reaches R38.2
- net 23_B: now also J12.1 (Pin_1); no longer J4.T
- net 29_B: now reaches J12.10 (Pin_10)
- net 29_B: now also R27.1
- net 30_B: now reaches J12.5 (Pin_5)
- net 30_B: now also U1.3 (Q0)
- net 31_B: now reaches J12.6 (Pin_6)
- net 31_B: now also U1.2 (Q1)
- net 32_B: now reaches J12.7 (Pin_7)
- net 32_B: now also U1.4 (Q2)
- net 33_B: now reaches J12.8 (Pin_8)
- net 33_B: now also U1.7 (Q3)
- net 34_B: now reaches J12.9 (Pin_9)
- net 34_B: now also U1.10 (Q4)
Other:
- note added: "3"
- note added: "4"
- moved on the sheet: D2, D4, D5, J1, J2, J3, J4, Q4, R23, R24, R25, R26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

Commit message: first testrun
Parts:
- added R99: 0, Resistor_SMD:R_0201_0603Metric, symbol Device:R
Connections:
- new net: R99.1, R99.2
Changed lines of the file:
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@@
   (junction (at 279.4 154.94) (diameter 0) (color 0 0 0 0)
   )
+  (junction (at 17.78 86.36) (diameter 0) (color 0 0 0 0)
+  )
   (junction (at 187.96 58.42) (diameter 0) (color 0 0 0 0)
   )
@@
   )
   (junction (at 182.88 49.53) (diameter 0) (color 0 0 0 0)
-  )
-  (junction (at 19.05 86.36) (diameter 0) (color 0 0 0 0)
   )
   (junction (at 187.96 119.38) (diameter 0) (color 0 0 0 0)
@@
     (stroke (width 0) (type default))
   )
-  (wire (pts (xy 19.05 86.36) (xy 19.05 90.17))
+  (wire (pts (xy 17.78 86.36) (xy 17.78 88.9))
     (stroke (width 0) (type default))
   )
@@
     (stroke (width 0) (type default))
   )
+  (wire (pts (xy 17.78 86.36) (xy 19.05 86.36))
+    (stroke (width 0) (type default))
+  )
   (wire (pts (xy 124.46 34.29) (xy 129.54 34.29))
     (stroke (width 0) (type default))
@@
     (stroke (width 0) (type default))
   )
+  (wire (pts (xy -33.02 -13.97) (xy -35.56 -13.97))
+    (stroke (width 0) (type default))
+  )
   (wire (pts (xy 176.53 40.64) (xy 176.53 101.6))
     (stroke (width 0) (type default))
@@
     (stroke (width 0) (type default))
   )
+  (wire (pts (xy -35.56 -13.97) (xy -35.56 -6.35))
+    (stroke (width 0) (type default))
+  )
   (wire (pts (xy 68.58 36.83) (xy 72.39 36.83))
     (stroke (width 0) (type default))
@@
     (stroke (width 0) (type default))
   )
+  (wire (pts (xy 19.05 85.09) (xy 19.05 82.55))
+    (stroke (width 0) (type default))
+  )
   (wire (pts (xy 36.83 86.36) (xy 50.8 86.36))
     (stroke (width 0) (type default))
@@
     (stroke (width 0) (type default))
   )
+  (wire (pts (xy 17.78 88.9) (xy 19.05 88.9))
+    (stroke (width 0) (type default))
+  )
   (wire (pts (xy 19.05 101.6) (xy 39.37 101.6))
     (stroke (width 0) (type default))
@@
     (stroke (width 0) (type default))
   )
+  (wire (pts (xy -35.56 -6.35) (xy -33.02 -6.35))
+    (stroke (width 0) (type default))
+  )
   (wire (pts (xy 222.25 33.02) (xy 201.93 33.02))
     (stroke (width 0) (type default))
@@
     (stroke (width 0) (type default))
   )
+  (wire (pts (xy 19.05 88.9) (xy 19.05 90.17))
+    (stroke (width 0) (type default))
+  )
   (wire (pts (xy 64.77 133.35) (xy 69.85 133.35))
     (stroke (width 0) (type default))
@@
     (stroke (width 0) (type default))
   )
-  (wire (pts (xy 19.05 82.55) (xy 19.05 86.36))
+  (wire (pts (xy 17.78 85.09) (xy 17.78 86.36))
     (stroke (width 0) (type default))
   )
@@
   )
   (wire (pts (xy 269.24 107.95) (xy 273.05 107.95))
+    (stroke (width 0) (type default))
+  )
+  (wire (pts (xy 17.78 85.09) (xy 19.05 85.09))
     (stroke (width 0) (type default))
   )
@@
     )
   )
+  (global_label "GND" (shape input) (at 17.78 86.36 180) (fields_autoplaced)
+    (effects (font (size 1.27 1.27)) (justify right))
+    (property "Intersheetrefs" "${INTERSHEET_REFS}" (at 11.0037 86.36 0)
+      (effects (font (size 1.27 1.27)) (justify right) hide)
+    )
+    (property "Netclass" "GND" (at 17.78 88.5508 0)
+      (effects (font (size 1.27 1.27)) (justify right) hide)
+    )
+  )
   (global_label "21_T" (shape input) (at -80.01 139.7 0) (fields_autoplaced)
     (effects (font (size 1.27 1.27)) (justify left))
@@
     )
   )
-  (global_label "GND" (shape input) (at 19.05 86.36 180) (fields_autoplaced)
-    (effects (font (size 1.27 1.27)) (justify right))
-    (property "Intersheetrefs" "${INTERSHEET_REFS}" (at 12.2737 86.36 0)
-      (effects (font (size 1.27 1.27)) (justify right) hide)
-    )
-    (property "Netclass" "Power" (at 19.05 88.5508 0)
-      (effects (font (size 1.27 1.27)) (justify right) hide)
-    )
-  )
   (global_label "14_T" (shape input) (at -81.28 55.88 0) (fields_autoplaced)
     (effects (font (size 1.27 1.27)) (justify left))
@@
     )
   )
+  (symbol (lib_id "Device:R") (at -33.02 -10.16 0) (unit 1)
+    (in_bom yes) (on_board yes) (dnp no) (fields_autoplaced)
+    (property "Reference" "R99" (at -29.21 -10.795 0)
+      (effects (font (size 1.27 1.27)) (justify left))
+    )
+    (property "Value" "0" (at -29.21 -8.255 0)
+      (effects (font (size 1.27 1.27)) (justify left))
+    )
+    (property "Footprint" "Resistor_SMD:R_0201_0603Metric" (at -34.798 -10.16 90)
+      (effects (font (size 1.27 1.27)) hide)
+    )
+    (property "Datasheet" "~" (at -33.02 -10.16 0)
+      (effects (font (size 1.27 1.27)) hide)
+    )
+    (pin "1")
+    (pin "2")
+    (instances
+      (project "BABY_Kicad"
+        (path "/6e5591c0-e975-4777-8ec0-68f3cef07627"
+          (reference "R99") (unit 1)
+        )
+      )
+    )
+  )

Commit message: Fixes
Connections:
- net 11_T: now also SW7.5 (B); no longer SW7.2 (B)
- net 12_T: now also SW7.4 (A); no longer SW7.1 (A)
- net 13_T: now also SW7.1 (A); no longer SW7.4 (A)
- net 14_T: now also SW7.3 (C); no longer SW7.6 (C)
- net 24_T: now also SW6.5 (B); no longer SW6.2 (B)
- net 28_T: now also SW6.4 (A); no longer SW6.1 (A)
- net 29_T: now also SW6.1 (A); no longer SW6.4 (A)
- net 35_T: now also SW6.3 (C); no longer SW6.6 (C)
- new net: SW6.2 (B), SW6.6 (C)
- new net: SW7.2 (B), SW7.6 (C)
Changed lines of the file:
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@@
     (stroke (width 0) (type default))
   )
+  (wire (pts (xy 134.62 118.11) (xy 142.24 118.11))
+    (stroke (width 0) (type default))
+  )
   (wire (pts (xy 113.03 134.62) (xy 113.03 151.13))
     (stroke (width 0) (type default))
@@
     (stroke (width 0) (type default))
   )
-  (wire (pts (xy 134.62 118.11) (xy 142.24 118.11))
-    (stroke (width 0) (type default))
-  )
   (wire (pts (xy 280.67 111.76) (xy 280.67 107.95))
     (stroke (width 0) (type default))
@@
     )
   )
-  (symbol (lib_id "Switch:SW_DPDT_x2") (at 129.54 115.57 0) (unit 1)
-    (in_bom yes) (on_board yes) (dnp no) (fields_autoplaced)
-    (property "Reference" "SW6" (at 129.54 109.22 0)
-      (effects (font (size 1.27 1.27)))
-    )
-    (property "Value" "SW_DPDT_x2" (at 129.54 111.76 0)
-      (effects (font (size 1.27 1.27)))
-    )
-    (property "Footprint" "1_SynthFootprints:DPDT_Tayda" (at 129.54 115.57 0)
-      (effects (font (size 1.27 1.27)) hide)
-    )
-    (property "Datasheet" "~" (at 129.54 115.57 0)
-      (effects (font (size 1.27 1.27)) hide)
-    )
-    (pin "1")
-    (pin "2")
-    (pin "3")
-    (pin "4")
-    (pin "5")
-    (pin "6")
-    (instances
-      (project "BABY_Kicad"
-        (path "/6e5591c0-e975-4777-8ec0-68f3cef07627"
-          (reference "SW6") (unit 1)
-        )
-      )
-    )
-  )
-  (symbol (lib_id "Switch:SW_DPDT_x2") (at 270.51 125.73 0) (unit 2)
-    (in_bom yes) (on_board yes) (dnp no) (fields_autoplaced)
-    (property "Reference" "SW7" (at 270.51 119.38 0)
-      (effects (font (size 1.27 1.27)))
-    )
-    (property "Value" "SW_DPDT_x2" (at 270.51 121.92 0)
-      (effects (font (size 1.27 1.27)))
-    )
-    (property "Footprint" "1_SynthFootprints:DPDT_Tayda" (at 270.51 125.73 0)
-      (effects (font (size 1.27 1.27)) hide)
-    )
-    (property "Datasheet" "~" (at 270.51 125.73 0)
-      (effects (font (size 1.27 1.27)) hide)
-    )
-    (pin "1")
-    (pin "2")
-    (pin "3")
-    (pin "4")
-    (pin "5")
-    (pin "6")
-    (instances
-      (project "BABY_Kicad"
-        (path "/6e5591c0-e975-4777-8ec0-68f3cef07627"
-          (reference "SW7") (unit 2)
-        )
-      )
-    )
-  )
   (symbol (lib_id "Switch:SW_SPDT") (at 138.43 69.85 0) (unit 1)
     (in_bom yes) (on_board yes) (dnp no) (fields_autoplaced)
@@
     )
   )
+  (symbol (lib_id "Switch:SW_DPDT_x2") (at 129.54 115.57 0) (unit 2)
+    (in_bom yes) (on_board yes) (dnp no) (fields_autoplaced)
+    (property "Reference" "SW6" (at 129.54 109.22 0)
+      (effects (font (size 1.27 1.27)))
+    )
+    (property "Value" "SW_DPDT_x2" (at 129.54 111.76 0)
+      (effects (font (size 1.27 1.27)))
+    )
+    (property "Footprint" "1_SynthFootprints:DPDT_Tayda" (at 129.54 115.57 0)
+      (effects (font (size 1.27 1.27)) hide)
+    )
+    (property "Datasheet" "~" (at 129.54 115.57 0)
+      (effects (font (size 1.27 1.27)) hide)
+    )
+    (pin "1")
+    (pin "2")
+    (pin "3")
+    (pin "4")
+    (pin "5")
+    (pin "6")
+    (instances
+      (project "BABY_Kicad"
+        (path "/6e5591c0-e975-4777-8ec0-68f3cef07627"
+          (reference "SW6") (unit 2)
+        )
+      )
+    )
+  )
   (symbol (lib_id "Device:R_Potentiometer") (at 213.36 101.6 270) (mirror x) (unit 1)
     (in_bom yes) (on_board yes) (dnp no)
@@
     )
   )
+  (symbol (lib_id "Switch:SW_DPDT_x2") (at 270.51 125.73 0) (unit 1)
+    (in_bom yes) (on_board yes) (dnp no) (fields_autoplaced)
+    (property "Reference" "SW7" (at 270.51 119.38 0)
+      (effects (font (size 1.27 1.27)))
+    )
+    (property "Value" "SW_DPDT_x2" (at 270.51 121.92 0)
+      (effects (font (size 1.27 1.27)))
+    )
+    (property "Footprint" "1_SynthFootprints:DPDT_Tayda" (at 270.51 125.73 0)
+      (effects (font (size 1.27 1.27)) hide)
+    )
+    (property "Datasheet" "~" (at 270.51 125.73 0)
+      (effects (font (size 1.27 1.27)) hide)
+    )
+    (pin "1")
+    (pin "2")
+    (pin "3")
+    (pin "4")
+    (pin "5")
+    (pin "6")
+    (instances
+      (project "BABY_Kicad"
+        (path "/6e5591c0-e975-4777-8ec0-68f3cef07627"
+          (reference "SW7") (unit 1)
+        )
+      )
+    )
+  )
   (symbol (lib_id "4xxx:4017") (at 135.89 156.21 0) (unit 1)
     (in_bom yes) (on_board yes) (dnp no) (fields_autoplaced)
@@
     )
   )
+  (symbol (lib_id "Switch:SW_DPDT_x2") (at 147.32 118.11 0) (unit 1)
+    (in_bom yes) (on_board yes) (dnp no) (fields_autoplaced)
+    (property "Reference" "SW6" (at 147.32 111.76 0)
+      (effects (font (size 1.27 1.27)))
+    )
+    (property "Value" "SW_DPDT_x2" (at 147.32 114.3 0)
+      (effects (font (size 1.27 1.27)))
+    )
+    (property "Footprint" "1_SynthFootprints:DPDT_Tayda" (at 147.32 118.11 0)
+      (effects (font (size 1.27 1.27)) hide)
+    )
+    (property "Datasheet" "~" (at 147.32 118.11 0)
+      (effects (font (size 1.27 1.27)) hide)
+    )
+    (pin "1")
+    (pin "2")
+    (pin "3")
+    (pin "4")
+    (pin "5")
+    (pin "6")
+    (instances
+      (project "BABY_Kicad"
+        (path "/6e5591c0-e975-4777-8ec0-68f3cef07627"
+          (reference "SW6") (unit 1)
+        )
+      )
+    )
+  )
+  (symbol (lib_id "Switch:SW_DPDT_x2") (at 254 123.19 0) (unit 2)
+    (in_bom yes) (on_board yes) (dnp no) (fields_autoplaced)
+    (property "Reference" "SW7" (at 254 116.84 0)
+      (effects (font (size 1.27 1.27)))
+    )
+    (property "Value" "SW_DPDT_x2" (at 254 119.38 0)
+      (effects (font (size 1.27 1.27)))
+    )
+    (property "Footprint" "1_SynthFootprints:DPDT_Tayda" (at 254 123.19 0)
+      (effects (font (size 1.27 1.27)) hide)
+    )
+    (property "Datasheet" "~" (at 254 123.19 0)
+      (effects (font (size 1.27 1.27)) hide)
+    )
+    (pin "1")
+    (pin "2")
+    (pin "3")
+    (pin "4")
+    (pin "5")
+    (pin "6")
+    (instances
+      (project "BABY_Kicad"
+        (path "/6e5591c0-e975-4777-8ec0-68f3cef07627"
+          (reference "SW7") (unit 2)
+        )
+      )
+    )
+  )
   (symbol (lib_id "power:PWR_FLAG") (at 67.31 93.98 180) (unit 1)
     (in_bom yes) (on_board yes) (dnp no) (fields_autoplaced)
@@
         )
       )
-    )
-  )
-  (symbol (lib_id "Switch:SW_DPDT_x2") (at 147.32 118.11 0) (unit 2)
-    (in_bom yes) (on_board yes) (dnp no) (fields_autoplaced)
-    (property "Reference" "SW6" (at 147.32 111.76 0)
-      (effects (font (size 1.27 1.27)))
-    )
-    (property "Value" "SW_DPDT_x2" (at 147.32 114.3 0)
-      (effects (font (size 1.27 1.27)))
-    )
-    (property "Footprint" "1_SynthFootprints:DPDT_Tayda" (at 147.32 118.11 0)
-      (effects (font (size 1.27 1.27)) hide)
-    )
-    (property "Datasheet" "~" (at 147.32 118.11 0)
-      (effects (font (size 1.27 1.27)) hide)
-    )
-    (pin "1")
-    (pin "2")
-    (pin "3")
-    (pin "4")
-    (pin "5")
-    (pin "6")
-    (instances
-      (project "BABY_Kicad"
-        (path "/6e5591c0-e975-4777-8ec0-68f3cef07627"
-          (reference "SW6") (unit 2)
-        )
-      )
-    )
-  )
-  (symbol (lib_id "Switch:SW_DPDT_x2") (at 254 123.19 0) (unit 1)
-    (in_bom yes) (on_board yes) (dnp no) (fields_autoplaced)
-    (property "Reference" "SW7" (at 254 116.84 0)
-      (effects (font (size 1.27 1.27)))
-    )
-    (property "Value" "SW_DPDT_x2" (at 254 119.38 0)
-      (effects (font (size 1.27 1.27)))
-    )
-    (property "Footprint" "1_SynthFootprints:DPDT_Tayda" (at 254 123.19 0)
-      (effects (font (size 1.27 1.27)) hide)
-    )
-    (property "Datasheet" "~" (at 254 123.19 0)
-      (effects (font (size 1.27 1.27)) hide)
-    )
-    (pin "1")
-    (pin "2")
-    (pin "3")
-    (pin "4")
-    (pin "5")
-    (pin "6")
-    (instances
-      (project "BABY_Kicad"
-        (path "/6e5591c0-e975-4777-8ec0-68f3cef07627"
-          (reference "SW7") (unit 1)
-        )
-      )
